Commit message: Visualize trajectory in 3d (needs cleanup)

File: obstacles.urdf (robot description, URDF)
Before this commit: robot office, 3 links, 2 joints
Links:
- added link obs3, mass .5; collision box size=1 1 2; visual box size=1 1 2
Joints:
- added joint obs3_to_ground: type fixed, parent ground, child obs3, origin xyz=0 0 0

Commit message: Augment obstacles with one extra obstacle

File: obstacles.urdf (robot description, URDF)
Before this commit: robot office, 4 links, 3 joints
Links:
- added link obs4, mass .5; collision box size=4 1 1; visual box size=4 1 1
Joints:
- added joint obs4_to_ground: type fixed, parent ground, child obs4, origin xyz=0 0 0

Commit message: Add obstacles back to sim

File: obstacles.urdf (robot description, URDF)
Before this commit: robot office, 5 links, 4 joints
Links:
- removed link obs4
Joints:
- removed joint obs4_to_ground
