Commit message: Create simulation test models

File: models/obstacles_walls.urdf (robot description, URDF)
Before this commit: robot office, 4 links, 3 joints
Links:
- added link obs4, mass .5; collision box size=4 0.4 1; visual box size=4 0.4 1
- link obs1: geometry collision box size=6 0.4 2; visual box size=6 0.4 2
- link obs2: geometry collision box size=6 0.4 2; visual box size=6 0.4 2
- link obs3: geometry collision box size=2 0.4 2; visual box size=2 0.4 2
Joints:
- added joint obs4_to_ground: type fixed, parent ground, child obs4, origin xyz=0 0 0
