Commit message: Add report

File: models/obstacles_forrest.urdf (robot description, URDF)
Before this commit: robot office, 7 links, 6 joints
Links:
- link ground: geometry collision box size=7 15 0.5; visual box size=7 15 0.5

File: models/obstacles_groups.urdf (robot description, URDF)
Before this commit: robot office, 18 links, 17 joints
Links:
- removed link obs5
- removed link obs7
- link ground: geometry collision box size=10 15 0.5; visual box size=10 15 0.5
Joints:
- removed joint obs5_to_ground
- removed joint obs7_to_ground

File: models/obstacles_walls.urdf (robot description, URDF)
Before this commit: robot office, 5 links, 4 joints
Links:
- link obs4: geometry collision box size=4 0.4 1.5; visual box size=4 0.4 1.5
